File: afc/schematics-v3/afc-xiao.kicad_pcb (KiCad board)
At the start: 2 copper layers, 110.5 x 59.7 mm, 14 parts

Commit message: updating schematic
Parts:
- moved C_1 13.1 mm to (174.6, 90.2)
- moved REF** 8.19 mm to (94.0, 125.6)
- moved REF** 8.19 mm to (94.0, 87.6)
- moved PWR 5.85 mm to (182.2, 108.0)
- moved FAN1 1.42 mm to (167.0, 82.5)
- moved ENV1 1.42 mm to (104.7, 110.5)
- moved FAN3 1.42 mm to (126.3, 82.5)
- moved FAN4 1.42 mm to (106.0, 82.5)
- moved C_2 1.42 mm to (154.3, 90.2)
- moved C_3 1.42 mm to (134.0, 90.2)
- moved XIAO-ESP32S3 1.42 mm to (130.2, 113.0)
- moved FAN2 1.42 mm to (146.7, 82.5)
- moved C_4 1.42 mm to (112.4, 90.2)
- moved C_E 1.42 mm to (146.7, 105.5)
Routing:
- net GND: track 0.00 -> 260.4 mm
- net TACHO2: track 85.2 -> 65.9 mm
- net TACHO1: track 80.1 -> 62.3 mm
- net PWM2: track 79.4 -> 61.6 mm
- net PWM1: track 74.3 -> 58.0 mm
- net 12V: track 153.8 -> 140.4 mm
- net 5V: track 53.2 -> 46.6 mm
- removed copper zone on F.Cu, net GND
Other:
- board size 110.5 x 59.7 mm -> 101.6 x 57.1 mm
